Commit message: revisiiii husky

File: install/husky_custom_description/share/husky_custom_description/urdf/custom_description.urdf.xacro (robot description, xacro)
@@ -25,24 +25,6 @@
   <xacro:arg name="ur5_enabled" default="$(optenv HUSKY_UR5_ENABLED false)" />
   <xacro:arg name="kinect_enabled" default="false" />
-  <xacro:include filename="$(find husky_description)/urdf/husky.urdf.xacro" />
-  <xacro:husky_robot />
+  <!-- <xacro:include filename="$(find husky_custom_description)/urdf/husky.urdf.xacro" /> -->
+  <!-- <xacro:husky_robot /> -->
   <!-- Insert customization below, sample provided: -->
-  <link name="bowler_link">
-    <visual>
-      <geometry>
-        <mesh filename="package://husky_custom_description/meshes/red_bowler.dae" />
-      </geometry>
-    </visual>
-    <collision>
-      <origin xyz="0 0 0.07" rpy="0 0 0" />
-      <geometry>
-        <box size="0.32 0.25 0.14" rpy="0 0 0"/>
-      </geometry>
-    </collision>
-  </link>
-  <joint name="bowler_joint" type="fixed">
-    <parent link="top_plate_link" />
-    <child link="bowler_link" />
-    <origin xyz="0.1 -0.1 0" rpy="0 0 0.5" />
-  </joint>
 </robot>

File: install/yolobot_description/share/yolobot_description/robot/husky_with_cameras.xacro (robot description, xacro)
@@ -3,4 +3,6 @@
   <!-- Include Husky base from husky_customization -->
   <xacro:include filename="$(find husky_custom_description)/urdf/custom_description.urdf.xacro"/>
+  <xacro:include filename="$(find husky_custom_description)/urdf/husky.urdf.xacro"/>
+  <!-- <xacro:husky_robot/> -->
   <!-- 1. Box Jetson Orin (paling bawah tower, warna hitam) -->
   <link name="orin_box_link">
