Commit message: Update huskybot_description

File: src/huskybot_description/robot/huskybot.urdf.xacro (robot description, xacro)
@@ -3,4 +3,42 @@
   <!-- Include Husky base dari package husky_description -->
   <xacro:include filename="$(find husky_description)/urdf/husky.urdf.xacro"/>  <!-- Import base Husky agar semua link/joint dasar tersedia -->
+  <!-- ==================== PLUGIN GAZEBO ==================== -->
+  <gazebo>
+    <plugin filename="libgazebo_ros_control.so" name="gazebo_ros_control"> <!-- Plugin ros2_control untuk integrasi controller ROS2 -->
+      <robotNamespace>/huskybot</robotNamespace>                          <!-- Namespace ROS robot (harus konsisten dengan node kontrol) -->
+      <robotParam>/robot_description</robotParam>                         <!-- Param robot_description (untuk robot_state_publisher) -->
+      <robotSimType>gazebo_ros_control/DefaultRobotHWSim</robotSimType>   <!-- Tipe hardware simulation Gazebo -->
+    </plugin>
+  </gazebo>
+  <gazebo>
+    <plugin filename="libgazebo_ros_diff_drive.so" name="differential_drive_controller"> <!-- Plugin diff_drive untuk cmd_vel dan odom -->
+      <ros>
+        <namespace>/huskybot</namespace>                                 <!-- Namespace ROS robot -->
+      </ros>
+      <left_joint>joint_right_wheel</left_joint>                         <!-- Joint kiri (cek urutan di base) -->
+      <right_joint>joint_left_wheel</right_joint>                        <!-- Joint kanan (cek urutan di base) -->
+      <wheel_separation>0.1</wheel_separation>                           <!-- Jarak antar roda (cek real robot) -->
+      <wheel_diameter>0.025</wheel_diameter>                             <!-- Diameter roda (cek real robot) -->
+      <max_wheel_torque>0.1</max_wheel_torque>                           <!-- Torsi maksimum roda -->
+      <max_wheel_acceleration>1.0</max_wheel_acceleration>               <!-- Akselerasi maksimum roda -->
+      <publish_odom>true</publish_odom>                                  <!-- Publish odometry ke ROS -->
+      <publish_odom_tf>true</publish_odom_tf>                            <!-- Publish TF odometry -->
+      <odometry_frame>odom</odometry_frame>                              <!-- Nama frame odometry -->
+      <robot_base_frame>chassis</robot_base_frame>                       <!-- Nama frame base robot -->
+    </plugin>
+  </gazebo>
+  <gazebo>
+    <plugin filename="libgazebo_ros_imu.so" name="gazebo_ros_imu_controller"> <!-- Plugin IMU -->
+      <robotNamespace>/huskybot/</robotNamespace>                        <!-- Namespace ROS robot -->
+      <topicName>imu/data3</topicName>                                  <!-- Topic output IMU -->
+      <serviceName>imu/service</serviceName>                            <!-- Nama service IMU -->
+      <bodyName>chassis</bodyName>                                      <!-- Link tempat IMU dipasang -->
+      <gaussianNoise>0</gaussianNoise>                                  <!-- Noise IMU (0 = tanpa noise) -->
+      <rpyOffsets>0 0 0</rpyOffsets>                                    <!-- Offset rotasi IMU -->
+      <updateRate>50.0</updateRate>                                     <!-- Frekuensi update IMU -->
+      <alwaysOn>true</alwaysOn>                                         <!-- IMU selalu aktif -->
+    </plugin>
+  </gazebo>
+  <!-- ==================== TOWER 3 TINGKAT ==================== -->
   <!-- 1. Box Jetson Orin (paling bawah tower, warna hitam) -->
   <link name="orin_box_link">  <!-- Link untuk box Jetson Orin -->
@@ -16,12 +54,12 @@
     <collision>
       <geometry>
-        <box size="0.25 0.18 0.09"/>  <!-- Dimensi collision sama dengan visual -->
+        <box size="0.25 0.18 0.09"/>
       </geometry>
       <origin xyz="0.0 0 0.045" rpy="0 0 0"/>
     </collision>
     <inertial>
-      <mass value="2.0"/>  <!-- Massa box -->
+      <mass value="2.0"/>
       <origin xyz="0.0 0 0.045"/>
-      <inertia ixx="0.02" ixy="0" ixz="0" iyy="0.02" iyz="0" izz="0.02"/>  <!-- Inersia sederhana -->
+      <inertia ixx="0.02" ixy="0" ixz="0" iyy="0.02" iyz="0" izz="0.02"/>
     </inertial>
   </link>
@@ -31,33 +69,61 @@
     <origin xyz="0 0 0.03" rpy="0 0 0"/>
   </joint>
-  <!-- 2. Tower Hexagonal (prisma segi enam, warna hitam) -->
-  <link name="hex_tower_link">
-    <visual>
-      <geometry>
-        <mesh filename="package://huskybot_description/meshes/hexagonal-prism.stl" scale="0.22 0.22 0.38"/>  <!-- Mesh tower -->
+  <!-- 2. Tower Hexagonal Bawah (prisma segi enam, warna hitam, tingkat 1) -->
+  <link name="hex_tower_lower_link">
+    <visual>
+      <geometry>
+        <mesh filename="package://huskybot_description/meshes/hexagonal-prism.stl" scale="0.22 0.22 0.18"/>
       </geometry>
       <material name="black">
         <color rgba="0 0 0 1"/>
       </material>
-      <origin xyz="0 0 0.07" rpy="0 0 0"/>
-    </visual>
-    <collision>
-      <geometry>
-        <mesh filename="package://huskybot_description/meshes/hexagonal-prism.stl" scale="0.22 0.22 0.38"/>
-      </geometry>
-      <origin xyz="0 0 0.07" rpy="0 0 0"/>
-    </collision>
-    <inertial>
-      <mass value="1.0"/>
-      <origin xyz="0 0 0.07"/>
-      <inertia ixx="0.01" ixy="0" ixz="0" iyy="0.01" iyz="0" izz="0.01"/>
-    </inertial>
-  </link>
-  <joint name="hex_tower_joint" type="fixed">
+      <origin xyz="0 0 0.09" rpy="0 0 0"/>
+    </visual>
+    <collision>
+      <geometry>
+        <mesh filename="package://huskybot_description/meshes/hexagonal-prism.stl" scale="0.22 0.22 0.18"/>
+      </geometry>
+      <origin xyz="0 0 0.09" rpy="0 0 0"/>
+    </collision>
+    <inertial>
+      <mass value="0.7"/>
+      <origin xyz="0 0 0.09"/>
+      <inertia ixx="0.007" ixy="0" ixz="0" iyy="0.007" iyz="0" izz="0.007"/>
+    </inertial>
+  </link>
+  <joint name="hex_tower_lower_joint" type="fixed">
     <parent link="orin_box_link"/>
-    <child link="hex_tower_link"/>
-    <origin xyz="0 0 0.07" rpy="0 0 0"/>
-  </joint>
-  <!-- 3. Tatakan Silinder LiDAR (warna hitam) -->
+    <child link="hex_tower_lower_link"/>
+    <origin xyz="0 0 0.09" rpy="0 0 0"/>
+  </joint>
+  <!-- 3. Tower Hexagonal Atas (prisma segi enam, warna hitam, tingkat 2) -->
+  <link name="hex_tower_upper_link">
+    <visual>
+      <geometry>
+        <mesh filename="package://huskybot_description/meshes/hexagonal-prism.stl" scale="0.18 0.18 0.18"/>
+      </geometry>
+      <material name="black">
+        <color rgba="0 0 0 1"/>
+      </material>
+      <origin xyz="0 0 0.09" rpy="0 0 0"/>
+    </visual>
+    <collision>
+      <geometry>
+        <mesh filename="package://huskybot_description/meshes/hexagonal-prism.stl" scale="0.18 0.18 0.18"/>
+      </geometry>
+      <origin xyz="0 0 0.09" rpy="0 0 0"/>
+    </collision>
+    <inertial>
+      <mass value="0.5"/>
+      <origin xyz="0 0 0.09"/>
+      <inertia ixx="0.005" ixy="0" ixz="0" iyy="0.005" iyz="0" izz="0.005"/>
+    </inertial>
+  </link>
+  <joint name="hex_tower_upper_joint" type="fixed">
+    <parent link="hex_tower_lower_link"/>
+    <child link="hex_tower_upper_link"/>
+    <origin xyz="0 0 0.18" rpy="0 0 0"/>
+  </joint>
+  <!-- 4. Tatakan Silinder LiDAR (paling atas tower, warna hitam, tingkat 3) -->
   <link name="lidar_base_link">
     <visual>
@@ -68,5 +134,5 @@
         <color rgba="0 0 0 1"/>
       </material>
-      <origin xyz="0 0 0.21" rpy="0 0 0"/>
+      <origin xyz="0 0 0.11" rpy="0 0 0"/>
     </visual>
     <collision>
@@ -74,18 +140,18 @@
         <cylinder length="0.04" radius="0.09"/>
       </geometry>
-      <origin xyz="0 0 0.21" rpy="0 0 0"/>
+      <origin xyz="0 0 0.11" rpy="0 0 0"/>
     </collision>
     <inertial>
       <mass value="0.5"/>
-      <origin xyz="0 0 0.21"/>
+      <origin xyz="0 0 0.11"/>
       <inertia ixx="0.005" ixy="0" ixz="0" iyy="0.005" iyz="0" izz="0.005"/>
     </inertial>
   </link>
   <joint name="lidar_base_joint" type="fixed">
-    <parent link="hex_tower_link"/>
+    <parent link="hex_tower_upper_link"/>
     <child link="lidar_base_link"/>
-    <origin xyz="0 0 0.19" rpy="0 0 0"/>
-  </joint>
-  <!-- 4. Velodyne VLP-32C (simulasi, gunakan mesh realistik jika ada) -->
+    <origin xyz="0 0 0.18" rpy="0 0 0"/>
+  </joint>
+  <!-- 5. Velodyne VLP-32C (paling atas) -->
   <link name="velodyne_link">
     <visual>
@@ -152,4 +218,5 @@
     </sensor>
   </gazebo>
+  <!-- ==================== KAMERA HEXAGONAL ==================== -->
   <!-- Macro untuk kamera di sisi tower heksagonal -->
   <xacro:macro name="hex_camera" params="idx yaw_deg">
@@ -164,7 +231,12 @@
         <origin xyz="0 0 0" rpy="0 0 0"/>
       </visual>
+      <inertial>
+        <mass value="0.1"/>
+        <origin xyz="0 0 0"/>
+        <inertia ixx="0.0001" ixy="0" ixz="0" iyy="0.0001" iyz="0" izz="0.0001"/>
+      </inertial>
     </link>
     <joint name="camera_${idx}_joint" type="fixed">
-      <parent link="hex_tower_link"/>
+      <parent link="hex_tower_upper_link"/>
       <child link="camera_${idx}_link"/>
       <origin xyz="${0.11 * cos(yaw_deg * 3.14159 / 180)} ${0.11 * sin(yaw_deg * 3.14159 / 180)} 0.09"
@@ -191,5 +263,5 @@
         <plugin name="gazebo_ros_camera" filename="libgazebo_ros_camera.so">
           <camera_name>camera_${idx}</camera_name>
-          <image_topic_name>image_raw</image_topic_name>
+          <image_topic_name>image_raw</image_topic_name> <!-- Topic kamera konsisten -->
           <camera_info_topic_name>camera_info</camera_info_topic_name>
           <frame_name>camera_${idx}_link</frame_name>

Commit message: Update 17 Mei 2025 12.35 WIB

File: src/huskybot_description/robot/huskybot.urdf.xacro (robot description, xacro)
@@ -13,24 +13,24 @@
   </gazebo>
   <!-- ==================== TAG ros2_control (WAJIB) ==================== -->
-  <ros2_control name="GazeboSystem" type="system">
+  <ros2_control name="GazeboSystem" type="system"> <!-- Tag ros2_control untuk integrasi dengan ros2_control dan controller_manager -->
     <hardware>
-      <plugin>gazebo_ros2_control/GazeboSystem</plugin>
+      <plugin>gazebo_ros2_control/GazeboSystem</plugin> <!-- Plugin hardware simulation Gazebo -->
     </hardware>
-    <joint name="front_left_wheel_joint">
+    <joint name="front_left_wheel_joint"> <!-- Joint roda kiri depan -->
+      <command_interface name="velocity"/> <!-- Interface kontrol kecepatan -->
+      <state_interface name="position"/> <!-- Interface baca posisi -->
+      <state_interface name="velocity"/> <!-- Interface baca kecepatan -->
+    </joint>
+    <joint name="front_right_wheel_joint"> <!-- Joint roda kanan depan -->
       <command_interface name="velocity"/>
       <state_interface name="position"/>
       <state_interface name="velocity"/>
     </joint>
-    <joint name="front_right_wheel_joint">
+    <joint name="rear_left_wheel_joint"> <!-- Joint roda kiri belakang -->
       <command_interface name="velocity"/>
       <state_interface name="position"/>
       <state_interface name="velocity"/>
     </joint>
-    <joint name="rear_left_wheel_joint">
-      <command_interface name="velocity"/>
-      <state_interface name="position"/>
-      <state_interface name="velocity"/>
-    </joint>
-    <joint name="rear_right_wheel_joint">
+    <joint name="rear_right_wheel_joint"> <!-- Joint roda kanan belakang -->
       <command_interface name="velocity"/>
       <state_interface name="position"/>
@@ -308,10 +308,10 @@
   </xacro:macro>
   <!-- Instantiate 6 cameras di sisi tower heksagonal (0, 60, 120, 180, 240, 300 derajat) -->
-  <xacro:hex_camera idx="front"    yaw_deg="0"/>
-  <xacro:hex_camera idx="front_left"  yaw_deg="60"/>
-  <xacro:hex_camera idx="left"     yaw_deg="120"/>
-  <xacro:hex_camera idx="rear"     yaw_deg="180"/>
-  <xacro:hex_camera idx="rear_right"  yaw_deg="240"/>
-  <xacro:hex_camera idx="right"    yaw_deg="300"/>
+  <xacro:hex_camera idx="front"    yaw_deg="0"/> <!-- Kamera depan -->
+  <xacro:hex_camera idx="front_left"  yaw_deg="60"/> <!-- Kamera depan kiri -->
+  <xacro:hex_camera idx="left"     yaw_deg="120"/> <!-- Kamera kiri -->
+  <xacro:hex_camera idx="rear"     yaw_deg="180"/> <!-- Kamera belakang -->
+  <xacro:hex_camera idx="rear_right"  yaw_deg="240"/> <!-- Kamera belakang kanan -->
+  <xacro:hex_camera idx="right"    yaw_deg="300"/> <!-- Kamera kanan -->
   <!--
     Kalibrasi extrinsic kamera-LiDAR:

Commit message: jjkahfauthatlj

File: src/huskybot_description/robot/huskybot.urdf.xacro (robot description, xacro)
@@ -2,35 +2,42 @@
 <robot xmlns:xacro="http://ros.org/wiki/xacro" name="husky_with_cameras"> <!-- Root elemen robot, pakai Xacro, nama robot unik -->
   <!-- ==================== INCLUDE BASE HUSKY ==================== -->
-  <xacro:include filename="$(find husky_description)/urdf/husky.urdf.xacro"/> <!-- Import base Husky agar semua link/joint dasar tersedia -->
+  <!-- Import base Husky agar semua link/joint dasar tersedia -->
+  <xacro:include filename="$(find husky_description)/urdf/husky.urdf.xacro"/> <!-- Pastikan package husky_description sudah di-build dan path benar -->
   <!-- ==================== PLUGIN GAZEBO ==================== -->
   <gazebo>
-    <plugin filename="libgazebo_ros2_control.so" name="gazebo_ros_control"> <!-- Plugin ros2_control untuk integrasi controller ROS2 -->
+    <!-- Plugin ros2_control untuk integrasi controller ROS2 -->
+    <plugin filename="libgazebo_ros2_control.so" name="gazebo_ros_control">
       <robotNamespace>/huskybot</robotNamespace> <!-- Namespace ROS robot (harus konsisten dengan node kontrol di huskybot_control) -->
       <robotParam>/robot_description</robotParam> <!-- Param robot_description (untuk robot_state_publisher) -->
       <robotSimType>gazebo_ros_control/DefaultRobotHWSim</robotSimType> <!-- Tipe hardware simulation Gazebo -->
-      <!-- Error handling: pastikan plugin sudah di-build dan path sudah di-export ke $GAZEBO_PLUGIN_PATH -->
+      <!-- ERROR HANDLING: Pastikan plugin sudah di-build dan path sudah di-export ke $GAZEBO_PLUGIN_PATH -->
     </plugin>
   </gazebo>
   <!-- ==================== TAG ros2_control (WAJIB) ==================== -->
-  <ros2_control name="GazeboSystem" type="system"> <!-- Tag ros2_control untuk integrasi dengan ros2_control dan controller_manager -->
+  <!-- Tag ros2_control untuk integrasi dengan ros2_control dan controller_manager -->
+  <ros2_control name="GazeboSystem" type="system">
     <hardware>
       <plugin>gazebo_ros2_control/GazeboSystem</plugin> <!-- Plugin hardware simulation Gazebo -->
     </hardware>
-    <joint name="front_left_wheel_joint"> <!-- Joint roda kiri depan -->
+    <!-- Joint roda kiri depan -->
+    <joint name="front_left_wheel_joint">
       <command_interface name="velocity"/> <!-- Interface kontrol kecepatan -->
       <state_interface name="position"/> <!-- Interface baca posisi -->
       <state_interface name="velocity"/> <!-- Interface baca kecepatan -->
     </joint>
-    <joint name="front_right_wheel_joint"> <!-- Joint roda kanan depan -->
+    <!-- Joint roda kanan depan -->
+    <joint name="front_right_wheel_joint">
       <command_interface name="velocity"/>
       <state_interface name="position"/>
       <state_interface name="velocity"/>
     </joint>
-    <joint name="rear_left_wheel_joint"> <!-- Joint roda kiri belakang -->
+    <!-- Joint roda kiri belakang -->
+    <joint name="rear_left_wheel_joint">
       <command_interface name="velocity"/>
       <state_interface name="position"/>
       <state_interface name="velocity"/>
     </joint>
-    <joint name="rear_right_wheel_joint"> <!-- Joint roda kanan belakang -->
+    <!-- Joint roda kanan belakang -->
+    <joint name="rear_right_wheel_joint">
       <command_interface name="velocity"/>
       <state_interface name="position"/>
@@ -39,4 +46,5 @@
   </ros2_control>
   <!-- ==================== SENSOR IMU ==================== -->
+  <!-- Sensor IMU pada link imu_link -->
   <gazebo reference="imu_link">
     <sensor type="imu" name="imu_sensor">
@@ -49,8 +57,10 @@
         <frame_name>imu_link</frame_name> <!-- Nama frame IMU -->
         <topicName>imu/data</topicName> <!-- Topic IMU di ROS2 -->
+        <!-- ERROR HANDLING: Pastikan plugin sudah di-build dan path sudah di-export ke $GAZEBO_PLUGIN_PATH -->
       </plugin>
     </sensor>
   </gazebo>
   <!-- ==================== SENSOR GPS ==================== -->
+  <!-- Sensor GPS pada link gps_link -->
   <!--
     ERROR HANDLING:
@@ -70,4 +80,5 @@
         <topicName>gps/fix</topicName> <!-- Topic GPS fix -->
         <velocityTopicName>gps/vel</velocityTopicName> <!-- Topic GPS velocity -->
+        <!-- ERROR HANDLING: Pastikan plugin sudah di-build dan path sudah di-export ke $GAZEBO_PLUGIN_PATH -->
       </plugin>
     </sensor>
@@ -82,19 +93,19 @@
     <visual>
       <geometry>
+        <box size="0.25 0.18 0.09"/> <!-- Ukuran box Jetson Orin -->
+      </geometry>
+      <material name="black">
+        <color rgba="0 0 0 1"/> <!-- Warna hitam -->
+      </material>
+      <origin xyz="0.0 0 0.045" rpy="0 0 0"/> <!-- Posisi box -->
+    </visual>
+    <collision>
+      <geometry>
         <box size="0.25 0.18 0.09"/>
       </geometry>
-      <material name="black">
-        <color rgba="0 0 0 1"/>
-      </material>
       <origin xyz="0.0 0 0.045" rpy="0 0 0"/>
-    </visual>
-    <collision>
-      <geometry>
-        <box size="0.25 0.18 0.09"/>
-      </geometry>
-      <origin xyz="0.0 0 0.045" rpy="0 0 0"/>
-    </collision>
-    <inertial>
-      <mass value="2.0"/>
+    </collision>
+    <inertial>
+      <mass value="2.0"/> <!-- Massa box -->
       <origin xyz="0.0 0 0.045"/>
       <inertia ixx="0.02" ixy="0" ixz="0" iyy="0.02" iyz="0" izz="0.02"/>
@@ -102,5 +113,5 @@
   </link>
   <joint name="orin_box_joint" type="fixed">
-    <parent link="top_plate_link"/>
+    <parent link="top_plate_link"/> <!-- Hubungkan ke top_plate_link dari base Husky -->
     <child link="orin_box_link"/>
     <origin xyz="0 0 0.03" rpy="0 0 0"/>
@@ -110,5 +121,5 @@
     <visual>
       <geometry>
-        <mesh filename="package://huskybot_description/meshes/hexagonal-prism.stl" scale="0.22 0.22 0.18"/>
+        <mesh filename="package://huskybot_description/meshes/hexagonal-prism.stl" scale="0.22 0.22 0.18"/> <!-- Mesh tower bawah -->
       </geometry>
       <material name="black">
@@ -138,5 +149,5 @@
     <visual>
       <geometry>
-        <mesh filename="package://huskybot_description/meshes/hexagonal-prism.stl" scale="0.18 0.18 0.18"/>
+        <mesh filename="package://huskybot_description/meshes/hexagonal-prism.stl" scale="0.18 0.18 0.18"/> <!-- Mesh tower atas -->
       </geometry>
       <material name="black">
@@ -166,5 +177,5 @@
     <visual>
       <geometry>
-        <cylinder length="0.04" radius="0.09"/>
+        <cylinder length="0.04" radius="0.09"/> <!-- Tatakan silinder LiDAR -->
       </geometry>
       <material name="black">
@@ -194,5 +205,5 @@
     <visual>
       <geometry>
-        <mesh filename="package://huskybot_description/meshes/velodyne_vlp32c.dae" scale="1 1 1"/>
+        <mesh filename="package://huskybot_description/meshes/velodyne_vlp32c.dae" scale="1 1 1"/> <!-- Mesh Velodyne -->
       </geometry>
       <material name="grey">
@@ -252,4 +263,5 @@
         <topicName>/velodyne_points</topicName>
         <frameName>velodyne_link</frameName>
+        <!-- ERROR HANDLING: Pastikan plugin sudah di-build dan path sudah di-export ke $GAZEBO_PLUGIN_PATH -->
       </plugin>
     </sensor>
@@ -261,5 +273,5 @@
       <visual>
         <geometry>
-          <mesh filename="package://huskybot_description/meshes/arducam_imx477.dae" scale="1 1 1"/>
+          <mesh filename="package://huskybot_description/meshes/arducam_imx477.dae" scale="1 1 1"/> <!-- Mesh kamera -->
         </geometry>
         <material name="black">
@@ -277,4 +289,5 @@
       <parent link="hex_tower_upper_link"/>
       <child link="camera_${idx}_link"/>
+      <!-- Posisi kamera di sisi tower heksagonal -->
       <origin xyz="${0.11 * cos(yaw_deg * 3.14159 / 180)} ${0.11 * sin(yaw_deg * 3.14159 / 180)} 0.09"
               rpy="0 0 ${yaw_deg * 3.14159 / 180}"/>
@@ -303,4 +316,5 @@
           <camera_info_topic_name>camera_info</camera_info_topic_name>
           <frame_name>camera_${idx}_link</frame_name>
+          <!-- ERROR HANDLING: Pastikan plugin sudah di-build dan path sudah di-export ke $GAZEBO_PLUGIN_PATH -->
         </plugin>
       </sensor>
@@ -323,4 +337,5 @@
         data: [ ... 16 nilai matriks ... ]
     Dokumentasikan transformasi ini di README dan gunakan untuk fusion 2D-3D.
+    ERROR HANDLING: Pastikan file YAML kalibrasi sudah ada dan path benar, jika tidak node fusion akan error.
   -->
 </robot>
