Commit message: Add huskybot_msgs

File: src/husky/husky_description/urdf/husky.urdf.xacro (robot description, xacro)
@@ -21,9 +21,9 @@
 ARISING IN ANY WAY OUT OF THE USE OF THIS SOFTWARE, EVEN IF ADVISED OF THE POSSIBILITY OF SUCH DAMAGE.
 -->
-<robot name="husky" xmlns:xacro="http://ros.org/wiki/xacro">
-  <!-- ==================== ARGUMEN XACRO (OOP) ==================== -->
-  <xacro:arg name="imu_xyz" default="$(optenv HUSKY_IMU_XYZ 0.19 0 0.149)"/>
-  <xacro:arg name="imu_rpy" default="$(optenv HUSKY_IMU_RPY 0 -1.5708 3.1416)"/>
-  <xacro:arg name="imu_parent" default="$(optenv HUSKY_IMU_PARENT base_link)"/>
+<robot name="husky" xmlns:xacro="http://ros.org/wiki/xacro"> <!-- Root elemen robot, nama unik -->
+  <!-- ==================== ARGUMEN XACRO (FULL OOP) ==================== -->
+  <xacro:arg name="imu_xyz" default="$(optenv HUSKY_IMU_XYZ 0.19 0 0.149)"/> <!-- Posisi IMU relatif parent -->
+  <xacro:arg name="imu_rpy" default="$(optenv HUSKY_IMU_RPY 0 -1.5708 3.1416)"/> <!-- Orientasi IMU -->
+  <xacro:arg name="imu_parent" default="$(optenv HUSKY_IMU_PARENT base_link)"/> <!-- Parent link IMU -->
   <xacro:arg name="laser_enabled" default="$(optenv HUSKY_LMS1XX_ENABLED 0)" />
   <xacro:arg name="laser_topic" default="$(optenv HUSKY_LMS1XX_TOPIC front/scan)"/>
@@ -108,4 +108,5 @@
   <xacro:arg name="outdoornav_configuration" default="$(optenv OUTDOORNAV_CONFIGURATION standard)" />
   <!-- ==================== INCLUDE MACRO & PROPERTY ==================== -->
+  <!-- Semua macro sensor dan dekorasi di-include agar bisa dipanggil OOP -->
   <xacro:include filename="$(find husky_description)/urdf/accessories/hokuyo_ust10.urdf.xacro"/>
   <xacro:include filename="$(find husky_description)/urdf/accessories/intel_realsense.urdf.xacro"/>
@@ -116,4 +117,6 @@
   <xacro:include filename="$(find husky_description)/urdf/decorations.urdf.xacro"/>
   <xacro:include filename="$(find husky_description)/urdf/wheel.urdf.xacro"/>
+  <!-- ==================== PROPERTY UKURAN & PARAMETER ==================== -->
+  <!-- Semua property ukuran dan parameter utama robot -->
   <xacro:property name="M_PI" value="3.14159"/>
   <xacro:property name="base_x_size" value="0.98740000"/>
@@ -126,9 +129,9 @@
   <xacro:property name="wheel_radius" value="0.1651"/>
   <!-- ==================== BASE LINK & FOOTPRINT ==================== -->
-  <link name="base_link">
+  <link name="base_link"> <!-- Link utama base robot -->
     <visual>
       <origin xyz="0 0 0" rpy="0 0 0"/>
       <geometry>
-        <mesh filename="package://husky_description/meshes/base_link.dae"/>
+        <mesh filename="package://husky_description/meshes/base_link.dae"/> <!-- Mesh visual base -->
       </geometry>
     </visual>
@@ -146,5 +149,5 @@
     </collision>
   </link>
-  <link name="base_footprint"/>
+  <link name="base_footprint"/> <!-- Link untuk navigasi 2D -->
   <joint name="base_footprint_joint" type="fixed">
     <origin xyz="0 0 ${wheel_vertical_offset - wheel_radius}" rpy="0 0 0"/>
@@ -166,4 +169,5 @@
   </joint>
   <!-- ==================== RODA (MACRO OOP) ==================== -->
+  <!-- Semua roda pakai macro agar OOP dan mudah diubah -->
   <xacro:husky_wheel wheel_prefix="front_left">
     <origin xyz="${wheelbase/2} ${track/2} ${wheel_vertical_offset}" rpy="0 0 0"/>
@@ -179,5 +183,5 @@
   </xacro:husky_wheel>
   <!-- ==================== DEKORASI ==================== -->
-  <xacro:husky_decorate/>
+  <xacro:husky_decorate/> <!-- Macro dekorasi visual -->
   <!-- ==================== SENSOR ARCH (OPSIONAL) ==================== -->
   <xacro:if value="$(arg sensor_arch)">
@@ -187,5 +191,5 @@
   </xacro:if>
   <!-- ==================== IMU (FULL OOP) ==================== -->
-  <link name="imu_link"/>
+  <link name="imu_link"/> <!-- Link IMU -->
   <joint name="imu_joint" type="fixed">
     <origin xyz="$(arg imu_xyz)" rpy="$(arg imu_rpy)"/>
@@ -229,4 +233,5 @@
   </xacro:if>
   <!-- ==================== REALSENSE & BLACKFLY (OOP, Macro) ==================== -->
+  <!-- Macro kamera, bisa diaktifkan via argumen -->
   <xacro:property name="realsense_enabled" value="$(arg realsense_enabled)"/>
   <xacro:property name="realsense_secondary_enabled" value="$(arg realsense_secondary_enabled)"/>
@@ -331,5 +336,5 @@
     </sensor>
   </gazebo>
-  <link name="gps_link"/>
+  <link name="gps_link"/> <!-- Link GPS, hanya boleh ada satu di seluruh workspace! -->
   <joint name="gps_joint" type="fixed">
     <parent link="base_link"/>

File: src/huskybot_description/robot/huskybot.urdf.xacro (robot description, xacro)
@@ -1,5 +1,5 @@
 <?xml version="1.0"?> <!-- Header XML wajib untuk file XML -->
 <robot xmlns:xacro="http://ros.org/wiki/xacro" name="husky_with_cameras"> <!-- Root elemen robot, pakai Xacro, nama robot unik -->
-  <!-- Include Husky base dari package husky_description -->
+  <!-- ==================== INCLUDE BASE HUSKY ==================== -->
   <xacro:include filename="$(find husky_description)/urdf/husky.urdf.xacro"/> <!-- Import base Husky agar semua link/joint dasar tersedia -->
   <!-- ==================== PLUGIN GAZEBO ==================== -->
@@ -32,5 +32,5 @@
     </plugin>
   </gazebo>
-  <!-- IMU ROS2 plugin -->
+  <!-- ==================== SENSOR IMU ==================== -->
   <gazebo reference="imu_link">
     <sensor type="imu" name="imu_sensor">
@@ -46,5 +46,11 @@
     </sensor>
   </gazebo>
-  <!-- GPS ROS2 plugin (tambahkan link gps_link di bawah jika belum ada) -->
+  <!-- ==================== SENSOR GPS ==================== -->
+  <!--
+    ERROR HANDLING:
+    - Jangan deklarasi ulang <link name="gps_link"/> dan joint jika sudah ada di base Husky!
+    - Jika ingin custom posisi, override joint dengan nama berbeda atau gunakan xacro argumen.
+    - Jika tetap ingin custom, pastikan hanya ada SATU link dengan nama gps_link di seluruh URDF!
+  -->
   <gazebo reference="gps_link">
     <sensor type="gps" name="gps_sensor">
@@ -61,11 +67,8 @@
     </sensor>
   </gazebo>
-  <!-- Link dan joint GPS (pastikan ada di URDF base, jika belum tambahkan di sini) -->
-  <link name="gps_link"/> <!-- Link GPS, posisi bisa diubah sesuai mounting -->
-  <joint name="gps_joint" type="fixed">
-    <parent link="base_link"/> <!-- Mount ke base_link -->
-    <child link="gps_link"/>
-    <origin xyz="0 0 0.3" rpy="0 0 0"/> <!-- Posisi GPS di atas robot -->
-  </joint>
+  <!--
+    <link name="gps_link"/> dan joint gps_joint DIHAPUS agar tidak duplikat!
+    Jika ingin custom mounting, edit di base Husky atau override dengan xacro argumen.
+  -->
   <!-- ==================== TOWER 3 TINGKAT ==================== -->
   <!-- 1. Box Jetson Orin (paling bawah tower, warna hitam) -->

Commit message: Update 15 Mei 2025 Subuh

File: src/husky/husky_description/urdf/husky.urdf.xacro (robot description, xacro)
@@ -314,14 +314,40 @@
     <xacro:outdoornav_sensors outdoornav_configuration="$(arg outdoornav_configuration)"/>
   </xacro:if>
-  <!-- ==================== PLUGIN CONTROLLER (ROS2) ==================== -->
+  <!-- ==================== TAG ros2_control (WAJIB) ==================== -->
+  <ros2_control name="GazeboSystem" type="system">
+    <hardware>
+      <plugin>gazebo_ros2_control/GazeboSystem</plugin>
+    </hardware>
+    <joint name="front_left_wheel_joint">
+      <command_interface name="velocity"/>
+      <state_interface name="position"/>
+      <state_interface name="velocity"/>
+    </joint>
+    <joint name="front_right_wheel_joint">
+      <command_interface name="velocity"/>
+      <state_interface name="position"/>
+      <state_interface name="velocity"/>
+    </joint>
+    <joint name="rear_left_wheel_joint">
+      <command_interface name="velocity"/>
+      <state_interface name="position"/>
+      <state_interface name="velocity"/>
+    </joint>
+    <joint name="rear_right_wheel_joint">
+      <command_interface name="velocity"/>
+      <state_interface name="position"/>
+      <state_interface name="velocity"/>
+    </joint>
+  </ros2_control>
+  <!-- ==================== PLUGIN GAZEBO (ros2_control) ==================== -->
   <!--
   <gazebo>
-    <plugin name="gazebo_ros_control" filename="libgazebo_ros2_control.so">
+    <plugin filename="libgazebo_ros2_control.so" name="gazebo_ros_control">
       <robotNamespace>$(arg robot_namespace)</robotNamespace>
-      <legacyModeNS>true</legacyModeNS>
+      <robotParam>/robot_description</robotParam>
+      <robotSimType>gazebo_ros_control/DefaultRobotHWSim</robotSimType>
     </plugin>
   </gazebo>
   -->
-  <!-- Plugin ros2_control DIHAPUS/DIKOMENTARI agar TIDAK DUPLIKAT dengan overlay huskybot.urdf.xacro -->
   <!-- ==================== PLUGIN GPS (REVISI: GANTI KE ROS2 NATIVE) ==================== -->
   <gazebo reference="gps_link">

File: src/huskybot_description/robot/huskybot.urdf.xacro (robot description, xacro)
@@ -12,24 +12,30 @@
     </plugin>
   </gazebo>
-  <gazebo>
-    <plugin filename="libgazebo_ros_diff_drive.so" name="differential_drive_controller"> <!-- Plugin diff_drive untuk cmd_vel dan odom -->
-      <ros>
-        <namespace>/huskybot</namespace> <!-- Namespace ROS robot, harus konsisten dengan node kontrol -->
-      </ros>
-      <left_joint>front_left_wheel</left_joint> <!-- Joint kiri depan -->
-      <left_joint>rear_left_wheel</left_joint> <!-- Joint kiri belakang -->
-      <right_joint>front_right_wheel</right_joint> <!-- Joint kanan depan -->
-      <right_joint>rear_right_wheel</right_joint> <!-- Joint kanan belakang -->
-      <wheel_separation>0.5708</wheel_separation> <!-- Jarak antar roda (track Husky, bisa di-xacro-kan) -->
-      <wheel_diameter>0.3302</wheel_diameter> <!-- Diameter roda (bisa di-xacro-kan) -->
-      <max_wheel_torque>0.1</max_wheel_torque> <!-- Torsi maksimum roda -->
-      <max_wheel_acceleration>1.0</max_wheel_acceleration> <!-- Akselerasi maksimum roda -->
-      <publish_odom>true</publish_odom> <!-- Publish odometry ke ROS -->
-      <publish_odom_tf>true</publish_odom_tf> <!-- Publish TF odometry -->
-      <odometry_frame>odom</odometry_frame> <!-- Nama frame odometry -->
-      <robot_base_frame>base_link</robot_base_frame> <!-- Nama frame base robot (Husky: base_link) -->
-      <!-- Error handling: pastikan semua joint di atas ada di URDF base Husky -->
-    </plugin>
-  </gazebo>
+  <!-- ==================== TAG ros2_control (WAJIB) ==================== -->
+  <ros2_control name="GazeboSystem" type="system">
+    <hardware>
+      <plugin>gazebo_ros2_control/GazeboSystem</plugin>
+    </hardware>
+    <joint name="front_left_wheel_joint">
+      <command_interface name="velocity"/>
+      <state_interface name="position"/>
+      <state_interface name="velocity"/>
+    </joint>
+    <joint name="front_right_wheel_joint">
+      <command_interface name="velocity"/>
+      <state_interface name="position"/>
+      <state_interface name="velocity"/>
+    </joint>
+    <joint name="rear_left_wheel_joint">
+      <command_interface name="velocity"/>
+      <state_interface name="position"/>
+      <state_interface name="velocity"/>
+    </joint>
+    <joint name="rear_right_wheel_joint">
+      <command_interface name="velocity"/>
+      <state_interface name="position"/>
+      <state_interface name="velocity"/>
+    </joint>
+  </ros2_control>
   <!-- ==================== SENSOR IMU ==================== -->
   <gazebo reference="imu_link">

Commit message: adlkfjakfjaesklfjasdlkfh

File: src/husky/husky_description/urdf/husky.urdf.xacro (robot description, xacro)
@@ -365,5 +365,27 @@
     </sensor>
   </gazebo>
-  <link name="gps_link"/> <!-- Link GPS, hanya boleh ada satu di seluruh workspace! -->
+  <!-- ==================== GPS LINK & JOINT ==================== -->
+  <link name="gps_link">
+    <visual>
+      <geometry>
+        <box size="0.05 0.05 0.02"/>
+      </geometry>
+      <material name="grey">
+        <color rgba="0.5 0.5 0.5 1"/>
+      </material>
+      <origin xyz="0 0 0.01" rpy="0 0 0"/>
+    </visual>
+    <collision>
+      <geometry>
+        <box size="0.05 0.05 0.02"/>
+      </geometry>
+      <origin xyz="0 0 0.01" rpy="0 0 0"/>
+    </collision>
+    <inertial>
+      <mass value="0.1"/>
+      <origin xyz="0 0 0.01"/>
+      <inertia ixx="0.0001" ixy="0" ixz="0" iyy="0.0001" iyz="0" izz="0.0001"/>
+    </inertial>
+  </link>
   <joint name="gps_joint" type="fixed">
     <parent link="base_link"/>

File: src/huskybot_description/robot/huskybot.urdf.xacro (robot description, xacro)
@@ -71,14 +71,13 @@
   <gazebo reference="gps_link">
     <sensor type="gps" name="gps_sensor">
-      <always_on>true</always_on> <!-- GPS selalu aktif -->
-      <update_rate>10</update_rate> <!-- Update rate GPS (Hz) -->
-      <plugin name="gps_sensor_plugin" filename="libgazebo_ros_gps_sensor.so"> <!-- Plugin GPS ROS2 native -->
+      <always_on>true</always_on>
+      <update_rate>10</update_rate>
+      <plugin name="gps_sensor_plugin" filename="libgazebo_ros_gps_sensor.so">
         <ros>
-          <namespace>/huskybot</namespace> <!-- Namespace ROS untuk topic GPS -->
+          <namespace>/huskybot</namespace>
         </ros>
-        <frame_name>gps_link</frame_name> <!-- Nama frame GPS -->
-        <topicName>gps/fix</topicName> <!-- Topic GPS fix -->
-        <velocityTopicName>gps/vel</velocityTopicName> <!-- Topic GPS velocity -->
-        <!-- ERROR HANDLING: Pastikan plugin sudah di-build dan path sudah di-export ke $GAZEBO_PLUGIN_PATH -->
+        <frame_name>gps_link</frame_name>
+        <topicName>gps/fix</topicName>
+        <velocityTopicName>gps/vel</velocityTopicName>
       </plugin>
     </sensor>
